File: hardware/capbank/varactor.kicad_sch (KiCad schematic)
At the start: 11 parts, among them U2 OPA2202IDR

Commit message: Small hardware changes
Parts:
- removed TP10: ~, TestPoint:TestPoint_THTPad_1.5x1.5mm_Drill0.7mm, symbol Connector:TestPoint
Changed lines of the file:
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@@
-	)
-	(junction
-		(at 104.14 92.71)
-		(diameter 0)
-		(color 0 0 0 0)
 	)
 	(junction
@@
 	(wire
 		(pts
-			(xy 97.79 92.71) (xy 104.14 92.71)
+			(xy 97.79 92.71) (xy 113.03 92.71)
 		)
 		(stroke
@@
 		(pts
 			(xy 172.72 85.09) (xy 175.26 85.09)
-		)
-		(stroke
-			(width 0)
-			(type default)
-		)
-	)
-	(wire
-		(pts
-			(xy 104.14 92.71) (xy 113.03 92.71)
 		)
 		(stroke
@@
 					(unit 1)
 				)
-			)
-		)
-	)
-	(symbol
-		(lib_id "Connector:TestPoint")
-		(at 104.14 92.71 0)
-		(unit 1)
-		(exclude_from_sim no)
-		(in_bom yes)
-		(on_board yes)
-		(dnp no)
-		(fields_autoplaced yes)
-		(property "Reference" "TP10"
-			(at 106.68 88.1379 0)
-			(effects
-				(font
-					(size 1.27 1.27)
-				)
-				(justify left)
-			)
-		)
-		(property "Value" "~"
-			(at 106.68 90.6779 0)
-			(effects
-				(font
-					(size 1.27 1.27)
-				)
-				(justify left)
-			)
-		)
-		(property "Footprint" "TestPoint:TestPoint_THTPad_1.5x1.5mm_Drill0.7mm"
-			(at 109.22 92.71 0)
-			(effects
-				(font
-					(size 1.27 1.27)
-				)
-				(hide yes)
-			)
-		)
-		(property "Datasheet" "~"
-			(at 109.22 92.71 0)
-			(effects
-				(font
-					(size 1.27 1.27)
-				)
-				(hide yes)
-			)
-		)
-		(property "Description" "test point"
-			(at 104.14 92.71 0)
-			(effects
-				(font
-					(size 1.27 1.27)
-				)
-				(hide yes)
-			)
-		)
-		(pin "1"
-		)
-		(instances
-			(project "capbank1"
-				(path "/461cb8a1-2d60-44a8-88b5-d61a3ba14a84/a75e6ab6-702b-4065-b99f-956a48aaae0a/9f6d23b6-b895-41cb-b038-be08ed2e2ab5"
-					(reference "TP10")
-					(unit 1)
-				)

Commit message: Add footprint for buffered-filter and replace pot with digital pot
Connections:
- net VBIAS_FB: now reaches R2.2, R3.2, U2.2 (-)
Changed lines of the file:
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@@
+		)
+	)
+	(label "VBIAS_FB"
+		(at 63.5 69.85 0)
+		(effects
+			(font
+				(size 1.27 1.27)
+			)
+			(justify left bottom)
 		)
 	)

Commit message: Update PCB with learned lessons
Parts:
- added R22: 1M, PCM_Resistor_SMD_AKL:R_0603_1608Metric, symbol Device:R
Connections:
- net VBIAS: now also R22.1; no longer R1.1
- new net: R1.1, R22.2
Changed lines of the file:
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@@
 	(text "Very large value, try 100k, 1M, 10M\nor use an inductor / choke.\nNote high values limit freq. agility"
 		(exclude_from_sim no)
-		(at 222.25 67.31 0)
+		(at 227.584 65.278 0)
 		(effects
 			(font
@@
 	(wire
 		(pts
+			(xy 201.93 57.15) (xy 201.93 62.23)
+		)
+		(stroke
+			(width 0)
+			(type default)
+		)
+	)
+	(wire
+		(pts
 			(xy 62.23 85.09) (xy 62.23 83.82)
 		)
@@
 	(wire
 		(pts
-			(xy 196.85 68.58) (xy 201.93 68.58)
+			(xy 196.85 57.15) (xy 201.93 57.15)
 		)
 		(stroke
@@
 	(wire
 		(pts
-			(xy 201.93 68.58) (xy 201.93 72.39)
-		)
-		(stroke
-			(width 0)
-			(type default)
-		)
-	)
-	(wire
-		(pts
 			(xy 22.86 34.29) (xy 22.86 33.02)
 		)
@@
 	(wire
 		(pts
+			(xy 201.93 69.85) (xy 201.93 72.39)
+		)
+		(stroke
+			(width 0)
+			(type default)
+		)
+	)
+	(wire
+		(pts
 			(xy 185.42 85.09) (xy 201.93 85.09)
 		)
@@
 	)
 	(label "VBIAS"
-		(at 196.85 68.58 0)
+		(at 196.85 57.15 0)
 		(effects
 			(font
@@
 					(unit 1)
 				)
+			)
+		)
+	)
+	(symbol
+		(lib_id "Device:R")
+		(at 201.93 66.04 0)
+		(unit 1)
+		(exclude_from_sim no)
+		(in_bom yes)
+		(on_board yes)
+		(dnp no)
+		(fields_autoplaced yes)
+		(property "Reference" "R22"
+			(at 204.47 64.7699 0)
+			(effects
+				(font
+					(size 1.27 1.27)
+				)
+				(justify left)
+			)
+		)
+		(property "Value" "1M"
+			(at 204.47 67.3099 0)
+			(effects
+				(font
+					(size 1.27 1.27)
+				)
+				(justify left)
+			)
+		)
+		(property "Footprint" "PCM_Resistor_SMD_AKL:R_0603_1608Metric"
+			(at 200.152 66.04 90)
+			(effects
+				(font
+					(size 1.27 1.27)
+				)
+				(hide yes)
+			)
+		)
+		(property "Datasheet" "~"
+			(at 201.93 66.04 0)
+			(effects
+				(font
+					(size 1.27 1.27)
+				)
+				(hide yes)
+			)
+		)
+		(property "Description" "Resistor"
+			(at 201.93 66.04 0)
+			(effects
+				(font
+					(size 1.27 1.27)
+				)
+				(hide yes)
+			)
+		)
+		(pin "1"
+		)
+		(pin "2"
+		)
+		(instances
+			(project "capbank1"
+				(path "/461cb8a1-2d60-44a8-88b5-d61a3ba14a84/a75e6ab6-702b-4065-b99f-956a48aaae0a/9f6d23b6-b895-41cb-b038-be08ed2e2ab5"
+					(reference "R22")
+					(unit 1)
+				)

Commit message: Various wiring fixes and add bleed resistor to antenna
Parts:
- added R20, R27, R28, R29, R30, R31: 22M, PCM_Resistor_SMD_AKL:R_0603_1608Metric, symbol Device:R
- C2: value 100n -> 100n (@32V)
Connections:
- net ANT1: now also R20.1
- net ANT2: now also R29.1
- net GND_ISOL: now also R28.2, R31.2
- new net: R20.2, R27.1
- new net: R27.2, R28.1
- new net: R29.2, R30.1
- new net: R30.2, R31.1
Other:
- note added: "50k on x2 DAC for 6x gain (5V * 6 = 30) 110k on x1 DAC for 12x gain (2.5V * 12 = 30)"
- note added: "8pF -> 120pF"
- note added: "Large value (try also 10 and 5Meg) just to allow charge to bleed, more than one to reduce the parasitic capacitance."
- moved on the sheet: C2

Commit message: Getting ready for manufacture
Parts:
- added C38: 80pF, PCM_Capacitor_SMD_AKL:C_0603_1608Metric, symbol Device:C
- R20, R27, R28, R29, R30, R31: value 22M -> 10M
Connections:
- net GND_ISOL: now also C38.1
- net at C11.1, D1.1 (K), D2.1 (K)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: now also C38.2
Other:
- note added: "BB639 x3: 8pF -> 120pF BB640 x2: 6pF -> 140pF BB640 x1: 3pF -> 70pF"
- note removed: "8pF -> 120pF"
Changed lines of the file:
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@@
 		)
 	)
-	(text "8pF -> 120pF"
-		(exclude_from_sim no)
-		(at 194.564 96.012 0)
+	(text "BB639 x3: 8pF -> 120pF\nBB640 x2: 6pF -> 140pF\nBB640 x1: 3pF -> 70pF"
+		(exclude_from_sim no)
+		(at 200.66 95.758 0)
 		(effects
 			(font
@@
 	)
 	(junction
+		(at 172.72 96.52)
+		(diameter 0)
+		(color 0 0 0 0)
+	)
+	(junction
 		(at 201.93 85.09)
 		(diameter 0)
@@
 	)
 	(junction
+		(at 185.42 96.52)
+		(diameter 0)
+		(color 0 0 0 0)
+	)
+	(junction
 		(at 97.79 92.71)
 		(diameter 0)
@@
 	(wire
 		(pts
+			(xy 182.88 110.49) (xy 185.42 110.49)
+		)
+		(stroke
+			(width 0)
+			(type default)
+		)
+	)
+	(wire
+		(pts
 			(xy 238.76 85.09) (xy 238.76 88.9)
 		)
@@
 	(wire
 		(pts
+			(xy 172.72 96.52) (xy 172.72 110.49)
+		)
+		(stroke
+			(width 0)
+			(type default)
+		)
+	)
+	(wire
+		(pts
 			(xy 157.48 102.87) (xy 157.48 85.09)
 		)
@@
 	(wire
 		(pts
+			(xy 185.42 110.49) (xy 185.42 96.52)
+		)
+		(stroke
+			(width 0)
+			(type default)
+		)
+	)
+	(wire
+		(pts
 			(xy 172.72 72.39) (xy 172.72 85.09)
 		)
@@
 		(pts
 			(xy 185.42 85.09) (xy 185.42 96.52)
+		)
+		(stroke
+			(width 0)
+			(type default)
+		)
+	)
+	(wire
+		(pts
+			(xy 172.72 110.49) (xy 175.26 110.49)
 		)
 		(stroke
@@
 			)
 		)
-		(property "Value" "22M"
+		(property "Value" "10M"
 			(at 139.7 102.8699 0)
 			(effects
@@
 			)
 		)
-		(property "Value" "22M"
+		(property "Value" "10M"
 			(at 241.3 93.9799 0)
 			(effects
@@
 			)
 		)
-		(property "Value" "22M"
+		(property "Value" "10M"
 			(at 241.3 111.7599 0)
 			(effects
@@
 			)
 		)
-		(property "Value" "22M"
+		(property "Value" "10M"
 			(at 139.7 93.9799 0)
 			(effects
@@
 			)
 		)
-		(property "Value" "22M"
+		(property "Value" "10M"
 			(at 139.7 111.7599 0)
 			(effects
@@
 			)
 		)
-		(property "Value" "22M"
+		(property "Value" "10M"
 			(at 241.3 102.8699 0)
 			(effects
@@
 					(unit 1)
 				)
+			)
+		)
+	)
+	(symbol
+		(lib_id "Device:C")
+		(at 179.07 110.49 90)
+		(unit 1)
+		(exclude_from_sim no)
+		(in_bom yes)
+		(on_board yes)
+		(dnp yes)
+		(fields_autoplaced yes)
+		(property "Reference" "C38"
+			(at 179.07 102.87 90)
+			(effects
+				(font
+					(size 1.27 1.27)
+				)
+			)
+		)
+		(property "Value" "80pF"
+			(at 179.07 105.41 90)
+			(effects
+				(font
+					(size 1.27 1.27)
+				)
+			)
+		)
+		(property "Footprint" "PCM_Capacitor_SMD_AKL:C_0603_1608Metric"
+			(at 182.88 109.5248 0)
+			(effects
+				(font
+					(size 1.27 1.27)
+				)
+				(hide yes)
+			)
+		)
+		(property "Datasheet" "~"
+			(at 179.07 110.49 0)
+			(effects
+				(font
+					(size 1.27 1.27)
+				)
+				(hide yes)
+			)
+		)
+		(property "Description" "Unpolarized capacitor"
+			(at 179.07 110.49 0)
+			(effects
+				(font
+					(size 1.27 1.27)
+				)
+				(hide yes)
+			)
+		)
+		(pin "1"
+		)
+		(pin "2"
+		)
+		(instances
+			(project "capbank1"
+				(path "/461cb8a1-2d60-44a8-88b5-d61a3ba14a84/a75e6ab6-702b-4065-b99f-956a48aaae0a/9f6d23b6-b895-41cb-b038-be08ed2e2ab5"
+					(reference "C38")
+					(unit 1)
+				)
