File: hardware/capbank/varactor.kicad_sch (KiCad schematic)
At the start: 18 parts, among them U2 OPA2202IDR

Commit message: Getting nearer to prod
Parts:
- C11, C12: value 10n -> 10n low esr
Changed lines of the file:
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@@
 	)
 	(rectangle
-		(start 171.45 64.135)
-		(end 186.055 99.695)
+		(start 170.18 64.135)
+		(end 186.69 102.87)
 		(stroke
 			(width 0)
@@
 			)
 		)
-		(property "Value" "10n"
+		(property "Value" "10n low esr"
 			(at 227.33 80.01 90)
 			(effects
@@
 			)
 		)
-		(property "Value" "10n"
+		(property "Value" "10n low esr"
 			(at 146.05 80.01 90)
 			(effects
