File: hardware/capbank/bias_supply.kicad_sch (KiCad schematic)
At the start: 27 parts, among them U12 LM317AEMP, U13 74HC14, U14 MCP1415, U15 MCP1415

Commit message: Small hardware changes
Parts:
- removed C18: 100n, PCM_Capacitor_SMD_AKL:C_0603_1608Metric, symbol Device:C
- removed unit 7 of U13
- added C1: 100n, PCM_Capacitor_SMD_AKL:C_0603_1608Metric, symbol Device:C
- added unit 6 of U13
- D4, D5, D6: value 1N5711 -> BAT46WJ; footprint Diode_THT:D_DO-35_SOD27_P7.62mm_Horizontal -> PCM_Diode_SMD_AKL:D_SOD-323
- D7: value 1N4007 -> 1N4007W; footprint Diode_THT:D_DO-35_SOD27_P7.62mm_Horizontal -> PCM_Diode_SMD_AKL:D_SOD-123
Connections:
- net GND_ISOL: now also U13.7 (GND), C1.2
- net OSC: now also U13.12; no longer U13.12
- net VDD_ISOL: now also U13.14 (VCC), C1.1
- net at C16.2, U13.10: now also U13.13; no longer U13.13
Other:
- note added: "VERIFIED oscillator"

Commit message: Add footprint for buffered-filter and replace pot with digital pot
Connections:
- net SWITCH_SUPPLY: now reaches C19.1, C20.1, C46.1, C47.1, D4.2 (A), FB1.2, U14.2 (Vdd), U15.2 (Vdd)
Changed lines of the file:
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@@
 	(wire
 		(pts
+			(xy 259.08 101.6) (xy 259.08 100.33)
+		)
+		(stroke
+			(width 0)
+			(type default)
+		)
+	)
+	(wire
+		(pts
 			(xy 107.95 87.63) (xy 107.95 105.41)
 		)
@@
 	(wire
 		(pts
+			(xy 259.08 72.39) (xy 259.08 74.93)
+		)
+		(stroke
+			(width 0)
+			(type default)
+		)
+	)
+	(wire
+		(pts
 			(xy 114.3 116.84) (xy 114.3 114.3)
 		)
@@
 		)
 	)
+	(label "SWITCH_SUPPLY"
+		(at 80.01 87.63 0)
+		(effects
+			(font
+				(size 1.27 1.27)
+			)
+			(justify left bottom)
+		)
+	)
 	(symbol
 		(lib_id "74xx:74HC14")
@@
 	(symbol
 		(lib_id "proj_power:VDD_ISOL")
-		(at 259.08 74.93 0)
+		(at 259.08 72.39 0)
 		(unit 1)
 		(exclude_from_sim no)
@@
 		(fields_autoplaced yes)
 		(property "Reference" "#PWR039"
-			(at 259.08 74.93 0)
+			(at 259.08 72.39 0)
 			(effects
 				(font
@@
 		)
 		(property "Value" "VDD_ISOL"
-			(at 259.08 69.85 0)
+			(at 259.08 67.31 0)
 			(effects
 				(font
@@
 		)
 		(property "Footprint" ""
-			(at 259.08 74.93 0)
+			(at 259.08 72.39 0)
 			(effects
 				(font
@@
 		)
 		(property "Datasheet" ""
-			(at 259.08 74.93 0)
+			(at 259.08 72.39 0)
 			(effects
 				(font
@@
 		)
 		(property "Description" ""
-			(at 259.08 74.93 0)
+			(at 259.08 72.39 0)
 			(effects
 				(font
@@
 	(symbol
 		(lib_id "proj_power:GND_ISOL")
-		(at 259.08 100.33 0)
+		(at 259.08 101.6 0)
 		(unit 1)
 		(exclude_from_sim no)
@@
 		(fields_autoplaced yes)
 		(property "Reference" "#PWR046"
-			(at 259.08 106.68 0)
+			(at 259.08 107.95 0)
 			(effects
 				(font
@@
 		)
 		(property "Value" "GND_ISOL"
-			(at 259.08 105.41 0)
+			(at 259.08 106.68 0)
 			(effects
 				(font
@@
 		)
 		(property "Footprint" ""
-			(at 259.08 100.33 0)
+			(at 259.08 101.6 0)
 			(effects
 				(font
@@
 		)
 		(property "Datasheet" ""
-			(at 259.08 100.33 0)
+			(at 259.08 101.6 0)
 			(effects
 				(font
@@
 		)
 		(property "Description" "Power symbol creates a global label with name \"GND_ISOL\" , isolated ground"
-			(at 259.08 100.33 0)
+			(at 259.08 101.6 0)
 			(effects
 				(font

Commit message: Some advances in pre-fabrication review
Parts:
- added R23: 7k, PCM_Resistor_SMD_AKL:R_1812_4532Metric, symbol Device:R
- R7: footprint PCM_Resistor_SMD_AKL:R_0603_1608Metric -> PCM_Resistor_SMD_AKL:R_1210_3225Metric_Pad1.30x2.65mm_HandSolder
Connections:
- net GND_ISOL: now also R23.2
- net HV_CLEAN: now also R23.1
Other:
- note added: "150mW"
- note added: "170mW"
- note added: "30.6V"
- note added: "7.7mW"
- note added: "Assumed 32V regulated for power worst-case"
- note added: "Resistor to ensure 10mA minimum load, We need 4.5mA additional (at most!) In practice, 3.5mA is enough, so may not need to be populated"
- note added: "V 5.5mA"
Changed lines of the file:
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@@
 		)
 	)
+	(text "30.6V"
+		(exclude_from_sim no)
+		(at 85.09 166.37 0)
+		(effects
+			(font
+				(size 1.27 1.27)
+			)
+		)
+	)
+	(text "150mW"
+		(exclude_from_sim no)
+		(at 153.924 159.004 0)
+		(effects
+			(font
+				(size 1.27 1.27)
+			)
+		)
+	)
 	(text "Oscillate under 10kHz for optimal \nripple rejection on LM317"
 		(exclude_from_sim no)
@@
 		)
 	)
+	(text "Assumed 32V regulated for power worst-case"
+		(exclude_from_sim no)
+		(at 109.474 147.574 0)
+		(effects
+			(font
+				(size 1.27 1.27)
+			)
+		)
+	)
+	(text "7.7mW"
+		(exclude_from_sim no)
+		(at 84.074 161.29 0)
+		(effects
+			(font
+				(size 1.27 1.27)
+			)
+		)
+	)
+	(text "Resistor to ensure 10mA minimum load, \nWe need 4.5mA additional (at most!)\n\nIn practice, 3.5mA is enough, so may not \nneed to be populated"
+		(exclude_from_sim no)
+		(at 183.134 154.94 0)
+		(effects
+			(font
+				(size 1.27 1.27)
+			)
+		)
+	)
+	(text "170mW"
+		(exclude_from_sim no)
+		(at 93.726 178.054 0)
+		(effects
+			(font
+				(size 1.27 1.27)
+			)
+		)
+	)
+	(text "V 5.5mA"
+		(exclude_from_sim no)
+		(at 92.202 154.94 0)
+		(effects
+			(font
+				(size 1.27 1.27)
+			)
+		)
+	)
 	(text "Caps sized for derating"
 		(exclude_from_sim no)
@@
 	)
 	(junction
+		(at 148.59 151.13)
+		(diameter 0)
+		(color 0 0 0 0)
+	)
+	(junction
 		(at 93.98 38.1)
 		(diameter 0)
@@
 	(wire
 		(pts
-			(xy 142.24 151.13) (xy 142.24 143.51)
+			(xy 152.4 151.13) (xy 152.4 142.24)
 		)
 		(stroke
@@
 	(wire
 		(pts
+			(xy 148.59 151.13) (xy 152.4 151.13)
+		)
+		(stroke
+			(width 0)
+			(type default)
+		)
+	)
+	(wire
+		(pts
 			(xy 93.98 60.96) (xy 93.98 63.5)
 		)
@@
 	(wire
 		(pts
-			(xy 133.35 151.13) (xy 142.24 151.13)
+			(xy 133.35 151.13) (xy 148.59 151.13)
 		)
 		(stroke
@@
 	)
 	(symbol
+		(lib_id "Device:R")
+		(at 148.59 154.94 0)
+		(unit 1)
+		(exclude_from_sim no)
+		(in_bom yes)
+		(on_board yes)
+		(dnp no)
+		(fields_autoplaced yes)
+		(property "Reference" "R23"
+			(at 151.13 153.6699 0)
+			(effects
+				(font
+					(size 1.27 1.27)
+				)
+				(justify left)
+			)
+		)
+		(property "Value" "7k"
+			(at 151.13 156.2099 0)
+			(effects
+				(font
+					(size 1.27 1.27)
+				)
+				(justify left)
+			)
+		)
+		(property "Footprint" "PCM_Resistor_SMD_AKL:R_1812_4532Metric"
+			(at 146.812 154.94 90)
+			(effects
+				(font
+					(size 1.27 1.27)
+				)
+				(hide yes)
+			)
+		)
+		(property "Datasheet" "~"
+			(at 148.59 154.94 0)
+			(effects
+				(font
+					(size 1.27 1.27)
+				)
+				(hide yes)
+			)
+		)
+		(property "Description" "Resistor"
+			(at 148.59 154.94 0)
+			(effects
+				(font
+					(size 1.27 1.27)
+				)
+				(hide yes)
+			)
+		)
+		(pin "2"
+		)
+		(pin "1"
+		)
+		(instances
+			(project "capbank1"
+				(path "/461cb8a1-2d60-44a8-88b5-d61a3ba14a84/ab1f86cc-d767-40d2-ba42-215e3d92336b"
+					(reference "R23")
+					(unit 1)
+				)
+			)
+		)
+	)
+	(symbol
 		(lib_id "Device:C_Polarized")
 		(at 73.66 173.99 0)
@@
 	)
 	(symbol
+		(lib_id "proj_power:GND_ISOL")
+		(at 148.59 158.75 0)
+		(unit 1)
+		(exclude_from_sim no)
+		(in_bom yes)
+		(on_board yes)
+		(dnp no)
+		(fields_autoplaced yes)
+		(property "Reference" "#PWR093"
+			(at 148.59 165.1 0)
+			(effects
+				(font
+					(size 1.27 1.27)
+				)
+				(hide yes)
+			)
+		)
+		(property "Value" "GND_ISOL"
+			(at 148.59 163.83 0)
+			(effects
+				(font
+					(size 1.27 1.27)
+				)
+			)
+		)
+		(property "Footprint" ""
+			(at 148.59 158.75 0)
+			(effects
+				(font
+					(size 1.27 1.27)
+				)
+				(hide yes)
+			)
+		)
+		(property "Datasheet" ""
+			(at 148.59 158.75 0)
+			(effects
+				(font
+					(size 1.27 1.27)
+				)
+				(hide yes)
+			)
+		)
+		(property "Description" "Power symbol creates a global label with name \"GND_ISOL\" , isolated ground"
+			(at 148.59 158.75 0)
+			(effects
+				(font
+					(size 1.27 1.27)
+				)
+				(hide yes)
+			)
+		)
+		(pin "1"
+		)
+		(instances
+			(project "capbank1"
+				(path "/461cb8a1-2d60-44a8-88b5-d61a3ba14a84/ab1f86cc-d767-40d2-ba42-215e3d92336b"
+					(reference "#PWR093")
+					(unit 1)
+				)
+			)
+		)
+	)
+	(symbol
 		(lib_id "PCM_Diode_Schottky_AKL:D_Schottky_Generic")
 		(at 52.07 38.1 0)
@@
 			)
 		)
-		(property "Footprint" "PCM_Resistor_SMD_AKL:R_0603_1608Metric"
+		(property "Footprint" "PCM_Resistor_SMD_AKL:R_1210_3225Metric_Pad1.30x2.65mm_HandSolder"
 			(at 87.122 173.99 90)
 			(effects
@@
 	(symbol
 		(lib_id "proj_power:HV_CLEAN")
-		(at 142.24 143.51 0)
+		(at 152.4 142.24 0)
 		(unit 1)
 		(exclude_from_sim no)
@@
 		(fields_autoplaced yes)
 		(property "Reference" "#PWR043"
-			(at 142.24 143.51 0)
+			(at 152.4 142.24 0)
 			(effects
 				(font
@@
 		)
 		(property "Value" "HV_CLEAN"
-			(at 142.24 138.43 0)
+			(at 152.4 137.16 0)
 			(effects
 				(font
@@
 		)
 		(property "Footprint" ""
-			(at 142.24 143.51 0)
+			(at 152.4 142.24 0)
 			(effects
 				(font
@@
 		)
 		(property "Datasheet" ""
-			(at 142.24 143.51 0)
+			(at 152.4 142.24 0)
 			(effects
 				(font
@@
 		)
 		(property "Description" ""
-			(at 142.24 143.51 0)
+			(at 152.4 142.24 0)
 			(effects
 				(font

Commit message: Various wiring fixes and add bleed resistor to antenna
Parts:
- C22: value 10u -> 10u (@32V)
- C45: value 100n -> 100n (@32V)
Other:
- moved on the sheet: C45, R23

Commit message: Getting ready for manufacture
Parts:
- removed U14, U15: MCP1415, Package_TO_SOT_SMD:SOT-23-5, symbol Driver_FET:MCP1415
- added R21: 2.8k, PCM_Resistor_SMD_AKL:R_1206_3216Metric_Pad1.30x1.75mm_HandSolder, symbol Device:R
- added R32: 3.3k, PCM_Resistor_SMD_AKL:R_1206_3216Metric_Pad1.30x1.75mm_HandSolder, symbol Device:R
- added U14, U15: FAN3111E, Package_TO_SOT_SMD:SOT-23-5, symbol Driver_FET:FAN3111E
- FB1: value Ferrite_Bead -> BLM18PG121SN1D
- R23: value 7k -> 3.3k; footprint PCM_Resistor_SMD_AKL:R_1812_4532Metric -> PCM_Resistor_SMD_AKL:R_1206_3216Metric_Pad1.30x1.75mm_HandSolder
- R7: value 5.6k -> 2.8k; footprint PCM_Resistor_SMD_AKL:R_1210_3225Metric_Pad1.30x2.65mm_HandSolder -> PCM_Resistor_SMD_AKL:R_1206_3216Metric_Pad1.30x1.75mm_HandSolder
Connections:
- net DRIVE: now also U14.5 (OUT)
- net GND_ISOL: now also R21.2, R32.2, U14.2 (GND), U15.2 (GND); no longer R23.2, R7.2
- net OSC: now also U15.3 (IN+)
- net SWITCH_SUPPLY: now also U14.1 (VDD), U15.1 (VDD)
- net VDD_ISOL: now also U14.4 (XREF), U15.4 (XREF)
- net ~{DRIVE}: now also U15.5 (OUT)
- net ~{OSC}: now also U14.3 (IN+)
- new net: R23.2, R32.1
- new net: R21.1, R7.2
Other:
- note added: "170mW, buying 2.7k"
- note removed: "170mW"

Commit message: Last review before prod
Parts:
- added D8: 1N4007W, PCM_Diode_SMD_AKL:D_SOD-123, symbol Device:D
Connections:
- net HV: now also D8.1 (K)
- net HV_CLEAN: now also D8.2 (A)
Changed lines of the file:
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@@
+	)
+	(junction
+		(at 63.5 151.13)
+		(diameter 0)
+		(color 0 0 0 0)
 	)
 	(junction
@@
 	(junction
 		(at 143.51 151.13)
+		(diameter 0)
+		(color 0 0 0 0)
+	)
+	(junction
+		(at 83.82 151.13)
 		(diameter 0)
 		(color 0 0 0 0)
@@
 	(wire
 		(pts
+			(xy 83.82 138.43) (xy 83.82 151.13)
+		)
+		(stroke
+			(width 0)
+			(type default)
+		)
+	)
+	(wire
+		(pts
 			(xy 44.45 115.57) (xy 50.8 115.57)
 		)
@@
 	(wire
 		(pts
-			(xy 59.69 151.13) (xy 66.04 151.13)
+			(xy 59.69 151.13) (xy 63.5 151.13)
 		)
 		(stroke
@@
 	(wire
 		(pts
+			(xy 83.82 151.13) (xy 88.9 151.13)
+		)
+		(stroke
+			(width 0)
+			(type default)
+		)
+	)
+	(wire
+		(pts
 			(xy 130.81 38.1) (xy 138.43 38.1)
 		)
@@
 	(wire
 		(pts
+			(xy 63.5 151.13) (xy 66.04 151.13)
+		)
+		(stroke
+			(width 0)
+			(type default)
+		)
+	)
+	(wire
+		(pts
 			(xy 156.21 43.18) (xy 156.21 29.21)
 		)
@@
 	(wire
 		(pts
+			(xy 69.85 138.43) (xy 63.5 138.43)
+		)
+		(stroke
+			(width 0)
+			(type default)
+		)
+	)
+	(wire
+		(pts
+			(xy 63.5 138.43) (xy 63.5 151.13)
+		)
+		(stroke
+			(width 0)
+			(type default)
+		)
+	)
+	(wire
+		(pts
 			(xy 107.95 105.41) (xy 114.3 105.41)
 		)
@@
 	(wire
 		(pts
+			(xy 77.47 138.43) (xy 83.82 138.43)
+		)
+		(stroke
+			(width 0)
+			(type default)
+		)
+	)
+	(wire
+		(pts
 			(xy 200.66 43.18) (xy 212.09 43.18)
 		)
@@
 	(wire
 		(pts
-			(xy 81.28 151.13) (xy 88.9 151.13)
+			(xy 81.28 151.13) (xy 83.82 151.13)
 		)
 		(stroke
@@
 					(unit 1)
 				)
+			)
+		)
+	)
+	(symbol
+		(lib_id "Device:D")
+		(at 73.66 138.43 0)
+		(unit 1)
+		(exclude_from_sim no)
+		(in_bom yes)
+		(on_board yes)
+		(dnp no)
+		(fields_autoplaced yes)
+		(property "Reference" "D8"
+			(at 73.66 132.08 0)
+			(effects
+				(font
+					(size 1.27 1.27)
+				)
+			)
+		)
+		(property "Value" "1N4007W"
+			(at 73.66 134.62 0)
+			(effects
+				(font
+					(size 1.27 1.27)
+				)
+			)
+		)
+		(property "Footprint" "PCM_Diode_SMD_AKL:D_SOD-123"
+			(at 73.66 138.43 0)
+			(effects
+				(font
+					(size 1.27 1.27)
+				)
+				(hide yes)
+			)
+		)
+		(property "Datasheet" "~"
+			(at 73.66 138.43 0)
+			(effects
+				(font
+					(size 1.27 1.27)
+				)
+				(hide yes)
+			)
+		)
+		(property "Description" "Diode"
+			(at 73.66 138.43 0)
+			(effects
+				(font
+					(size 1.27 1.27)
+				)
+				(hide yes)
+			)
+		)
+		(property "Sim.Device" "D"
+			(at 73.66 138.43 0)
+			(effects
+				(font
+					(size 1.27 1.27)
+				)
+				(hide yes)
+			)
+		)
+		(property "Sim.Pins" "1=K 2=A"
+			(at 73.66 138.43 0)
+			(effects
+				(font
+					(size 1.27 1.27)
+				)
+				(hide yes)
+			)
+		)
+		(pin "1"
+		)
+		(pin "2"
+		)
+		(instances
+			(project "capbank1"
+				(path "/461cb8a1-2d60-44a8-88b5-d61a3ba14a84/ab1f86cc-d767-40d2-ba42-215e3d92336b"
+					(reference "D8")
+					(unit 1)
+				)
