File: hardware/capbank/bias_supply.kicad_sch (KiCad schematic)
At the start: 31 parts, among them U12 LM317AEMP, U13 74HC14, U14 FAN3111E, U15 FAN3111E

Commit message: Small changes after building the PCB
Parts:
- C16: value 3.3n -> 1n
- R23, R32: now not fitted
Other:
- note added: "WRONG: It oscillates at roughly half the 1-gate frequency! Adjusted values for real build!"
Changed lines of the file:
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@@
 	(generator_version "9.0")
 	(paper "A4")
+	(text "WRONG: It oscillates at roughly half the 1-gate frequency! \nAdjusted values for real build!"
+		(exclude_from_sim no)
+		(at 233.934 24.892 0)
+		(effects
+			(font
+				(size 1.27 1.27)
+			)
+		)
+	)
 	(text "VERIFIED oscillator"
 		(exclude_from_sim no)
@@
 		(in_bom yes)
 		(on_board yes)
-		(dnp no)
+		(dnp yes)
 		(fields_autoplaced yes)
 		(property "Reference" "R23"
@@
 			)
 		)
-		(property "Value" "3.3n"
+		(property "Value" "1n"
 			(at 204.47 38.0999 0)
 			(effects
@@
 		(in_bom yes)
 		(on_board yes)
-		(dnp no)
+		(dnp yes)
 		(fields_autoplaced yes)
 		(property "Reference" "R32"
