File: hardware/capbank/capbank1.kicad_pcb (KiCad board)
At the start: 2 copper layers, 91 x 64 mm, 139 parts, among them J1 XY308-2P 2.54MM, J3 Conn_01x02, J4 Conn_01x02, J5 Conn_01x06, K1 3570.1333.121 COMUS, K2 3570.1333.121 COMUS, K4 3570.1333.121 COMUS, SW2 SW_SPST, U1 ULN2003, U10 TS861IL, U11 NXJ1S1212MC, U12 LM317AEMP, U13 74HC14, U14 FAN3111E, U15 FAN3111E, U16 LM78L05ACZ, U17 MCP4012-503ECH, U2 OPA2202IDR, U3 MCP1525-TO, U4 MCP4921-EP, U5 PAI130M61, U6 MCP6021T-E-OT, U7 74HC4046AD, U8 ATtiny84A-SS, U9 LM78L05ACZ, Y1 16MHz

Commit message: Last review before prod
Parts:
- added D8: 1N4007W, PCM_Diode_SMD_AKL:D_SOD-123, B.Cu at (131.8, 109.3)
- JP8: moved to B.Cu
- moved JP8 15.5 mm to (118.5, 61.0), turned to 0 degrees
Connections:
- JP8 pad 1: /Microcontroller/FSK_IN -> Net-(JP8-A)
- JP8 pad 2: /Microcontroller/FSK_DEMOD -> VDD
- U17 pad 6: VDD -> Net-(JP8-A)
- U8 pad 10: /Microcontroller/FSK_IN -> /Microcontroller/FSK_DEMOD
Routing:
- net /Microcontroller/FSK_IN: track 8.53 -> 0.00 mm
- net /Microcontroller/FSK_DEMOD: track 30.4 -> 37.8 mm
- net GND: track 75.9 -> 82.3 mm, vias 61 -> 64
- net HV_CLEAN: track 75.8 -> 81.6 mm, vias 2 -> 3
- net Net-(JP8-A): track 0.00 -> 3.10 mm, vias 0 -> 1
- net HV: track 26.4 -> 27.5 mm, vias 0 -> 1
- net /Isolated/ANT2: track 38.1 -> 39.0 mm
- net VDD: track 165.4 -> 165.0 mm, vias 2 -> 3
Other:
- board text added: "FSK"
- board text added: "FSK DEM"
