File: hardware/capbank/extsupply.kicad_sch (KiCad schematic)
At the start: 7 parts, among them U16 LM78L05ACZ

Commit message: Small hardware changes
Parts:
- removed C26: 10u, PCM_Capacitor_THT_AKL:CP_Radial_D5.0mm_P2.00mm, symbol Device:C_Polarized

Commit message: Some advances in pre-fabrication review
Parts:
- C30: value 100n -> 0.22u
Other:
- moved on the sheet: C31
Changed lines of the file:
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@@
+	)
+	(junction
+		(at 177.8 80.01)
+		(diameter 0)
+		(color 0 0 0 0)
 	)
 	(junction
@@
 		(color 0 0 0 0)
 	)
-	(junction
-		(at 187.96 80.01)
-		(diameter 0)
-		(color 0 0 0 0)
-	)
 	(wire
 		(pts
-			(xy 187.96 76.2) (xy 187.96 80.01)
+			(xy 177.8 76.2) (xy 177.8 80.01)
 		)
 		(stroke
@@
 	(wire
 		(pts
-			(xy 166.37 80.01) (xy 187.96 80.01)
+			(xy 166.37 80.01) (xy 177.8 80.01)
 		)
 		(stroke
@@
 			)
 		)
-		(property "Value" "100n"
+		(property "Value" "0.22u"
 			(at 144.78 85.0899 0)
 			(effects
@@
 	(symbol
 		(lib_id "power:GND")
-		(at 187.96 87.63 0)
+		(at 177.8 87.63 0)
 		(unit 1)
 		(exclude_from_sim no)
@@
 		(dnp no)
 		(property "Reference" "#PWR080"
-			(at 187.96 93.98 0)
+			(at 177.8 93.98 0)
 			(effects
 				(font
@@
 		)
 		(property "Value" "GND"
-			(at 187.96 92.71 0)
+			(at 177.8 92.71 0)
 			(effects
 				(font
@@
 		)
 		(property "Footprint" ""
-			(at 187.96 87.63 0)
+			(at 177.8 87.63 0)
 			(effects
 				(font
@@
 		)
 		(property "Datasheet" ""
-			(at 187.96 87.63 0)
+			(at 177.8 87.63 0)
 			(effects
 				(font
@@
 		)
 		(property "Description" "Power symbol creates a global label with name \"GND\" , ground"
-			(at 187.96 87.63 0)
+			(at 177.8 87.63 0)
 			(effects
 				(font
@@
 	(symbol
 		(lib_id "power:VDD")
-		(at 187.96 76.2 0)
+		(at 177.8 76.2 0)
 		(unit 1)
 		(exclude_from_sim no)
@@
 		(dnp no)
 		(property "Reference" "#PWR075"
-			(at 187.96 80.01 0)
+			(at 177.8 80.01 0)
 			(effects
 				(font
@@
 		)
 		(property "Value" "VDD"
-			(at 187.96 71.12 0)
+			(at 177.8 71.12 0)
 			(effects
 				(font
@@
 		)
 		(property "Footprint" ""
-			(at 187.96 76.2 0)
+			(at 177.8 76.2 0)
 			(effects
 				(font
@@
 		)
 		(property "Datasheet" ""
-			(at 187.96 76.2 0)
+			(at 177.8 76.2 0)
 			(effects
 				(font
@@
 		)
 		(property "Description" "Power symbol creates a global label with name \"VDD\""
-			(at 187.96 76.2 0)
+			(at 177.8 76.2 0)
 			(effects
 				(font
@@
 	(symbol
 		(lib_id "Device:C")
-		(at 187.96 83.82 0)
+		(at 177.8 83.82 0)
 		(unit 1)
 		(exclude_from_sim no)
@@
 		(fields_autoplaced yes)
 		(property "Reference" "C31"
-			(at 191.77 82.5499 0)
+			(at 181.61 82.5499 0)
 			(effects
 				(font
@@
 		)
 		(property "Value" "100n"
-			(at 191.77 85.0899 0)
+			(at 181.61 85.0899 0)
 			(effects
 				(font
@@
 		)
 		(property "Footprint" "PCM_Capacitor_SMD_AKL:C_0603_1608Metric"
-			(at 188.9252 87.63 0)
+			(at 178.7652 87.63 0)
 			(effects
 				(font
@@
 		)
 		(property "Datasheet" "~"
-			(at 187.96 83.82 0)
+			(at 177.8 83.82 0)
 			(effects
 				(font
@@
 		)
 		(property "Description" "Unpolarized capacitor"
-			(at 187.96 83.82 0)
-			(effects
-				(font
+			(at 177.8 83.82 0)
+			(effects
+				(font

Commit message: Getting ready for manufacture
Parts:
- C27: footprint PCM_Capacitor_THT_AKL:CP_Radial_D8.0mm_P3.50mm -> PCM_Capacitor_THT_AKL:CP_Radial_D6.3mm_P2.50mm
Changed lines of the file:
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@@
 			)
 		)
-		(property "Footprint" "PCM_Capacitor_THT_AKL:CP_Radial_D8.0mm_P3.50mm"
+		(property "Footprint" "PCM_Capacitor_THT_AKL:CP_Radial_D6.3mm_P2.50mm"
 			(at 63.1952 85.09 0)
 			(effects
