File: hardware/capbank/fsk_demod.kicad_sch (KiCad schematic)
At the start: 31 parts, among them U10 TS861IL, U18 MCP4013-xxxxCH, U6 MCP6021T-E-OT, U7 74HC4046AD

Commit message: Getting ready for manufacture
Other:
- note added: "Cheaper: TLV9061xDBV"
- note added: "Or CD74HC4046AM"
Changed lines of the file:
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@@
+		)
+	)
+	(text "Cheaper: TLV9061xDBV"
+		(exclude_from_sim no)
+		(at 81.026 180.594 0)
+		(effects
+			(font
+				(size 1.27 1.27)
+			)
 		)
 	)
@@
 		(effects
 			(font
+				(size 1.27 1.27)
+			)
+		)
+	)
+	(text "Or CD74HC4046AM"
+		(exclude_from_sim no)
+		(at 88.9 36.83 0)
+		(effects
+			(font

Commit message: Getting nearer to prod
Parts:
- removed U18: MCP4013-xxxxCH, Package_TO_SOT_SMD:SOT-23-6, symbol Potentiometer_Digital:MCP4013-xxxxCH
- added R33, R34: 50k, PCM_Resistor_SMD_AKL:R_0603_1608Metric, symbol Device:R
- added U17: MCP4012-503ECH, Package_TO_SOT_SMD:SOT-23-6, symbol Potentiometer_Digital:MCP4012-xxxxCH
Connections:
- net GND: now also R33.1, U17.2 (VSS)
- net RHEO_CS: now also U17.4 (~{CS})
- net RHEO_UD: now also U17.3 (U/~{D})
- net VDD: now also R34.2, U17.1 (VDD), U17.6 (A)
- net at R25.1: now also R33.2, R34.1, U17.5 (W)
Other:
- moved on the sheet: C26

Commit message: Last review before prod
Parts:
- added JP8: 0, PCM_Resistor_SMD_AKL:R_0603_1608Metric, symbol Jumper:Jumper_2_Small_Open
Connections:
- net VDD: now also JP8.2 (B); no longer U17.6 (A)
- new net: JP8.1 (A), U17.6 (A)
Changed lines of the file:
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@@
 	)
 	(junction
-		(at 191.77 121.92)
+		(at 63.5 161.29)
 		(diameter 0)
 		(color 0 0 0 0)
 	)
 	(junction
-		(at 63.5 161.29)
+		(at 191.77 121.92)
 		(diameter 0)
 		(color 0 0 0 0)
@@
 	(wire
 		(pts
-			(xy 191.77 137.16) (xy 191.77 121.92)
-		)
-		(stroke
-			(width 0)
-			(type default)
-		)
-	)
-	(wire
-		(pts
 			(xy 81.28 64.77) (xy 95.25 64.77)
 		)
@@
 	(wire
 		(pts
+			(xy 191.77 129.54) (xy 191.77 137.16)
+		)
+		(stroke
+			(width 0)
+			(type default)
+		)
+	)
+	(wire
+		(pts
 			(xy 191.77 121.92) (xy 191.77 120.65)
 		)
@@
 	(wire
 		(pts
+			(xy 191.77 121.92) (xy 191.77 124.46)
+		)
+		(stroke
+			(width 0)
+			(type default)
+		)
+	)
+	(wire
+		(pts
 			(xy 67.31 144.78) (xy 90.17 144.78)
 		)
@@
 					(unit 1)
 				)
+			)
+		)
+	)
+	(symbol
+		(lib_id "Jumper:Jumper_2_Small_Open")
+		(at 191.77 127 90)
+		(unit 1)
+		(exclude_from_sim no)
+		(in_bom yes)
+		(on_board yes)
+		(dnp no)
+		(fields_autoplaced yes)
+		(property "Reference" "JP8"
+			(at 193.04 125.7299 90)
+			(effects
+				(font
+					(size 1.27 1.27)
+				)
+				(justify right)
+			)
+		)
+		(property "Value" "0"
+			(at 193.04 128.2699 90)
+			(effects
+				(font
+					(size 1.27 1.27)
+				)
+				(justify right)
+			)
+		)
+		(property "Footprint" "PCM_Resistor_SMD_AKL:R_0603_1608Metric"
+			(at 191.77 127 0)
+			(effects
+				(font
+					(size 1.27 1.27)
+				)
+				(hide yes)
+			)
+		)
+		(property "Datasheet" "~"
+			(at 191.77 127 0)
+			(effects
+				(font
+					(size 1.27 1.27)
+				)
+				(hide yes)
+			)
+		)
+		(property "Description" "Jumper, 2-pole, small symbol, open"
+			(at 191.77 127 0)
+			(effects
+				(font
+					(size 1.27 1.27)
+				)
+				(hide yes)
+			)
+		)
+		(pin "1"
+		)
+		(pin "2"
+		)
+		(instances
+			(project "capbank1"
+				(path "/461cb8a1-2d60-44a8-88b5-d61a3ba14a84/d9c36704-5831-4033-b353-abc8255d1c86/9a2777cd-eff3-4d8b-a149-a95a84199cc5"
+					(reference "JP8")
+					(unit 1)
+				)

Commit message: Small changes after building the PCB
Parts:
- R13, R14: now not fitted
Changed lines of the file:
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@@
 		(in_bom yes)
 		(on_board yes)
-		(dnp no)
+		(dnp yes)
 		(fields_autoplaced yes)
 		(property "Reference" "R13"
@@
 		(in_bom yes)
 		(on_board yes)
-		(dnp no)
+		(dnp yes)
 		(fields_autoplaced yes)
 		(property "Reference" "R14"

Commit message: Updates
Parts:
- C40: value 120p -> 1n
- JP12, JP14, JP16, JP9: now not fitted
- R13: value 10k -> 220k; now fitted
- R14: value 10k -> 47k; now fitted
Changed lines of the file:
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@@
 		(in_bom yes)
 		(on_board yes)
-		(dnp no)
+		(dnp yes)
 		(fields_autoplaced yes)
 		(property "Reference" "JP12"
@@
 			)
 		)
-		(property "Value" "120p"
+		(property "Value" "1n"
 			(at 34.29 54.6099 0)
 			(effects
@@
 		(in_bom yes)
 		(on_board yes)
-		(dnp no)
+		(dnp yes)
 		(property "Reference" "JP16"
 			(at 86.36 43.18 0)
@@
 		(in_bom yes)
 		(on_board yes)
-		(dnp no)
+		(dnp yes)
 		(property "Reference" "JP14"
 			(at 78.74 67.056 0)
@@
 		(in_bom yes)
 		(on_board yes)
-		(dnp yes)
+		(dnp no)
 		(fields_autoplaced yes)
 		(property "Reference" "R13"
@@
 			)
 		)
-		(property "Value" "10k"
+		(property "Value" "220k"
 			(at 31.75 71.1199 0)
 			(effects
@@
 		(in_bom yes)
 		(on_board yes)
-		(dnp yes)
+		(dnp no)
 		(fields_autoplaced yes)
 		(property "Reference" "R14"
@@
 			)
 		)
-		(property "Value" "10k"
+		(property "Value" "47k"
 			(at 41.91 71.1199 0)
 			(effects
@@
 		(in_bom yes)
 		(on_board yes)
-		(dnp no)
+		(dnp yes)
 		(property "Reference" "JP9"
 			(at 34.29 140.97 0)

Commit message: Fix very stupid design mistake, now the comparator value is wider tunable
Required changing R33 to 2.7k
Parts:
- R33: value 50k -> 2.7k
Changed lines of the file:
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@@
 			)
 		)
-		(property "Value" "50k"
+		(property "Value" "2.7k"
 			(at 200.66 147.3199 0)
 			(effects
