File: hardware/capbank/isol_supply.kicad_sch (KiCad schematic)
At the start: 8 parts, among them U11 NXJ1S1212MC, U9 LM78L05ACZ

Commit message: Small hardware changes
Parts:
- removed C49: 10u, PCM_Capacitor_THT_AKL:CP_Radial_D5.0mm_P2.00mm, symbol Device:C_Polarized

Commit message: Some advances in pre-fabrication review
Parts:
- removed C14: 10u, PCM_Capacitor_THT_AKL:CP_Radial_D5.0mm_P2.00mm, symbol Device:C_Polarized
- added FB2: 82223C (22uH), proj_footprints:82223C, symbol PCM_Device_AKL:Ferrite_Bead
- added R24: 1.2k, PCM_Resistor_SMD_AKL:R_1206_3216Metric_Pad1.30x1.75mm_HandSolder, symbol Device:R
- C13: value 100n -> 4.7u; footprint PCM_Capacitor_SMD_AKL:C_0603_1608Metric -> Capacitor_SMD:C_1210_3225Metric_Pad1.33x2.70mm_HandSolder
- C23: value 100n -> 0.22u
Connections:
- net GND_ISOL: now also R24.2
- net V_SUPPLY_ISOL: now also FB2.2, R24.1; no longer U11.8 (+VOUT)
- new net: FB2.1, U11.8 (+VOUT)
Other:
- note added: "Minimum load is 10% of rated, so 8.3mA -> 100mW"
- note removed: "TODO: Add a ferrite / PI filter or something"
- moved on the sheet: C13, C25, C48

Commit message: Various wiring fixes and add bleed resistor to antenna
Changed lines of the file:
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@@
+	)
+	(junction
+		(at 229.87 88.9)
+		(diameter 0)
+		(color 0 0 0 0)
 	)
 	(junction
@@
 		(pts
 			(xy 41.91 95.25) (xy 52.07 95.25)
+		)
+		(stroke
+			(width 0)
+			(type default)
+		)
+	)
+	(wire
+		(pts
+			(xy 229.87 88.9) (xy 240.03 88.9)
 		)
 		(stroke
@@
 					(unit 1)
 				)
+			)
+		)
+	)
+	(symbol
+		(lib_id "power:PWR_FLAG")
+		(at 240.03 88.9 0)
+		(unit 1)
+		(exclude_from_sim no)
+		(in_bom yes)
+		(on_board yes)
+		(dnp no)
+		(fields_autoplaced yes)
+		(property "Reference" "#FLG04"
+			(at 240.03 86.995 0)
+			(effects
+				(font
+					(size 1.27 1.27)
+				)
+				(hide yes)
+			)
+		)
+		(property "Value" "PWR_FLAG"
+			(at 240.03 83.82 0)
+			(effects
+				(font
+					(size 1.27 1.27)
+				)
+			)
+		)
+		(property "Footprint" ""
+			(at 240.03 88.9 0)
+			(effects
+				(font
+					(size 1.27 1.27)
+				)
+				(hide yes)
+			)
+		)
+		(property "Datasheet" "~"
+			(at 240.03 88.9 0)
+			(effects
+				(font
+					(size 1.27 1.27)
+				)
+				(hide yes)
+			)
+		)
+		(property "Description" "Special symbol for telling ERC where power comes from"
+			(at 240.03 88.9 0)
+			(effects
+				(font
+					(size 1.27 1.27)
+				)
+				(hide yes)
+			)
+		)
+		(pin "1"
+		)
+		(instances
+			(project ""
+				(path "/461cb8a1-2d60-44a8-88b5-d61a3ba14a84/bb6379f6-afea-4713-b534-7575122a6ac9"
+					(reference "#FLG04")
+					(unit 1)
+				)
