File: hardware/capbank/mcu.kicad_sch (KiCad schematic)
At the start: 18 parts, among them J3 Conn_01x02, J4 Conn_01x02, J5 Conn_01x06, SW2 SW_SPST, U8 ATtiny84A-SS, Y1 16MHz

Commit message: Last review before prod
Parts:
- removed JP8: 0, PCM_Resistor_SMD_AKL:R_0603_1608Metric, symbol Jumper:Jumper_2_Small_Open
Connections:
- net FSK_IN is gone; now on net FSK_DEMOD: U8.10 (PA3)
Changed lines of the file:
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@@
-	(wire
-		(pts
-			(xy 257.81 36.83) (xy 270.51 36.83)
-		)
-		(stroke
-			(width 0)
-			(type default)
-		)
-	)
 	(wire
 		(pts
@@
 		(pts
 			(xy 50.8 57.15) (xy 58.42 57.15)
-		)
-		(stroke
-			(width 0)
-			(type default)
-		)
-	)
-	(wire
-		(pts
-			(xy 251.46 36.83) (xy 252.73 36.83)
 		)
 		(stroke
@@
 		)
 	)
-	(label "FSK_IN"
-		(at 251.46 36.83 180)
-		(effects
-			(font
-				(size 1.27 1.27)
-			)
-			(justify right bottom)
-		)
-	)
 	(label "SPI_SCK{slash}PRG_SCK"
 		(at 58.42 46.99 0)
@@
 		)
 	)
-	(label "FSK_IN"
+	(label "FSK_DEMOD"
 		(at 231.14 111.76 0)
 		(effects
@@
 	(label "~{RESET}"
 		(at 231.14 134.62 0)
-		(effects
-			(font
-				(size 1.27 1.27)
-			)
-			(justify left bottom)
-		)
-	)
-	(label "FSK_DEMOD"
-		(at 270.51 36.83 0)
 		(effects
 			(font
@@
 					(unit 1)
 				)
-			)
-		)
-	)
-	(symbol
-		(lib_id "Jumper:Jumper_2_Small_Open")
-		(at 255.27 36.83 0)
-		(unit 1)
-		(exclude_from_sim no)
-		(in_bom yes)
-		(on_board yes)
-		(dnp no)
-		(property "Reference" "JP8"
-			(at 255.016 47.244 0)
-			(effects
-				(font
-					(size 1.27 1.27)
-				)
-			)
-		)
-		(property "Value" "0"
-			(at 258.064 47.244 0)
-			(effects
-				(font
-					(size 1.27 1.27)
-				)
-			)
-		)
-		(property "Footprint" "PCM_Resistor_SMD_AKL:R_0603_1608Metric"
-			(at 255.27 36.83 0)
-			(effects
-				(font
-					(size 1.27 1.27)
-				)
-				(hide yes)
-			)
-		)
-		(property "Datasheet" "~"
-			(at 255.27 36.83 0)
-			(effects
-				(font
-					(size 1.27 1.27)
-				)
-				(hide yes)
-			)
-		)
-		(property "Description" "Jumper, 2-pole, small symbol, open"
-			(at 255.27 36.83 0)
-			(effects
-				(font
-					(size 1.27 1.27)
-				)
-				(hide yes)
-			)
-		)
-		(pin "1"
-		)
-		(pin "2"
-		)
-		(instances
-			(project "capbank1"
-				(path "/461cb8a1-2d60-44a8-88b5-d61a3ba14a84/d9c36704-5831-4033-b353-abc8255d1c86"
-					(reference "JP8")
-					(unit 1)
-				)

Commit message: Small changes after building the PCB
Parts:
- R10, R9: now not fitted
Changed lines of the file:
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@@
 		(in_bom yes)
 		(on_board yes)
-		(dnp no)
+		(dnp yes)
 		(fields_autoplaced yes)
 		(property "Reference" "R9"
@@
 		(in_bom yes)
 		(on_board yes)
-		(dnp no)
+		(dnp yes)
 		(fields_autoplaced yes)
 		(property "Reference" "R10"
