File: hardware/capbank/relays.kicad_sch (KiCad schematic)
At the start: 9 parts, among them K1 3570.1333.121 COMUS, K2 3570.1333.121 COMUS, K4 3570.1333.121 COMUS, U1 ULN2003

Commit message: Small hardware changes
Parts:
- removed TP2, TP3, TP4: ~, TestPoint:TestPoint_THTPad_1.5x1.5mm_Drill0.7mm, symbol Connector:TestPoint

Commit message: Various wiring fixes and add bleed resistor to antenna
Connections:
- net GND: now also U1.1 (I1), U1.2 (I2), U1.4 (I4), U1.6 (I6)
- no-connect marks 8 -> 4
Other:
- moved on the sheet: C32, C33
